Commit message: feat: robot_ip dynamic parameter + joint_trajectory_controller rename
- FairinoHardwareInterface reads robot_ip from URDF <ros2_control> hardware parameters
- Falls back to default 192.168.50.101 if not specified
- Renamed fairino5_controller -> joint_trajectory_controller for mf_manipulator compatibility
- Switched ros2_control xacro from mock to real FairinoHardwareInterface plugin

File: fairino5_v6_moveit2_config/config/fairino5_v6_robot.ros2_control.xacro (robot description, xacro)
@@ -1,10 +1,10 @@
 <?xml version="1.0"?>
 <robot xmlns:xacro="http://www.ros.org/wiki/xacro">
-    <xacro:macro name="fairino5_v6_robot_ros2_control" params="name initial_positions_file">
+    <xacro:macro name="fairino5_v6_robot_ros2_control" params="name initial_positions_file robot_ip:='192.168.50.101'">
         <xacro:property name="initial_positions" value="${load_yaml(initial_positions_file)['initial_positions']}"/>
         <ros2_control name="${name}" type="system">
             <hardware>
-                <!-- By default, set up controllers for simulation. This won't work on real hardware -->
-                <plugin>mock_components/GenericSystem</plugin>
+                <plugin>fairino_hardware/FairinoHardwareInterface</plugin>
+                <param name="robot_ip">${robot_ip}</param>
             </hardware>
             <joint name="j1">

Commit message: feat: add use_fake_hardware conditional to ros2_control xacro
Supports mock_components/GenericSystem when use_fake_hardware:=true,
matching mf_manipulator's fr5_v6.ros2_control.xacro pattern.

File: fairino5_v6_moveit2_config/config/fairino5_v6_robot.ros2_control.xacro (robot description, xacro)
@@ -1,10 +1,16 @@
 <?xml version="1.0"?>
 <robot xmlns:xacro="http://www.ros.org/wiki/xacro">
-    <xacro:macro name="fairino5_v6_robot_ros2_control" params="name initial_positions_file robot_ip:='192.168.50.101'">
+    <xacro:macro name="fairino5_v6_robot_ros2_control" params="name initial_positions_file robot_ip:='192.168.50.101' use_fake_hardware:=false">
         <xacro:property name="initial_positions" value="${load_yaml(initial_positions_file)['initial_positions']}"/>
         <ros2_control name="${name}" type="system">
             <hardware>
-                <plugin>fairino_hardware/FairinoHardwareInterface</plugin>
-                <param name="robot_ip">${robot_ip}</param>
+                <xacro:if value="${use_fake_hardware}">
+                    <plugin>mock_components/GenericSystem</plugin>
+                    <param name="state_following_offset">0.0</param>
+                </xacro:if>
+                <xacro:unless value="${use_fake_hardware}">
+                    <plugin>fairino_hardware/FairinoHardwareInterface</plugin>
+                    <param name="robot_ip">${robot_ip}</param>
+                </xacro:unless>
             </hardware>
             <joint name="j1">
